File: Teensy/PCB/ADSRModule/ADSRModule.kicad_pcb (KiCad board)
At the start: 2 copper layers, 53.3 x 106.7 mm, 41 parts, among them J1 Conn_02x03_Odd_Even, SW1 SW_SPDT_MSM, U1 Teensy4.0

Commit message: Fixed component names on schematic
Parts:
- J1: value Conn_02x03_Odd_Even -> Power_Connector_2x3
- RV1: value R_Potentiometer -> Decay_Time_Mod_Scale
- RV10: value R_Potentiometer -> Output_Scale
- RV11: value R_Potentiometer -> Sustain_Offset
- RV2: value R_Potentiometer -> Release_Time_Mod_Scale
- RV3: value R_Potentiometer -> Attack_Time_Mod_Scale
- RV4: value R_Potentiometer -> Attack_Slope
- RV5: value R_Potentiometer -> Decay_Time_Offset
- RV6: value R_Potentiometer -> Release_Slope
- RV7: value R_Potentiometer -> Release_Time_Offset
- RV8: value R_Potentiometer -> Decay_Slope
- RV9: value R_Potentiometer -> Attack_Time_Offset
- SW1: value SW_SPDT_MSM -> Mode_Switch
Connections:
- net /Input/Signal renamed /Attack_Time_Mod_In/Signal
- net /Input/Switch renamed /Attack_Time_Mod_In/Switch
- net /Input1/Signal renamed /Decay_Time_Mod_In/Signal
- net /Input1/Switch renamed /Decay_Time_Mod_In/Switch
- net /Input2/Signal renamed /Trigger_In/Signal
- net /Input2/Switch renamed /Trigger_In/Switch
- net /Input3/Signal renamed /Release_Time_Mod_In/Signal
- net /Input3/Switch renamed /Release_Time_Mod_In/Switch
- net /Output1/Signal renamed /Inverted_Output/Signal
- net /Output1/Switch renamed /Inverted_Output/Switch

Commit message: Replaced Schematic Lines with references
Connections:
- net /Attack_Time_Mod_In/Signal renamed /T7
- net /Decay_Time_Mod_In/Signal renamed /T15
- net /Inverted_Output/Signal renamed /T8
- net /Output/Signal renamed /T1
- net /Release_Time_Mod_In/Signal renamed /T16
- net /Trigger_In/Signal renamed /T0
- net Net-(RV1-Pad1) renamed /T9
- net Net-(RV1-Pad2) renamed /T21
- net Net-(RV10-Pad1) renamed /T11
- net Net-(RV10-Pad2) renamed /T23
- net Net-(RV11-Pad1) renamed /T6
- net Net-(RV11-Pad2) renamed /T20
- net Net-(RV2-Pad1) renamed /T29
- net Net-(RV2-Pad2) renamed /T25
- net Net-(RV3-Pad1) renamed /T3
- net Net-(RV3-Pad2) renamed /T17
- net Net-(RV4-Pad1) renamed /T2
- net Net-(RV4-Pad2) renamed /T14
- net Net-(RV5-Pad1) renamed /T10
- net Net-(RV5-Pad2) renamed /T22
- net Net-(RV6-Pad1) renamed /T27
- net Net-(RV6-Pad2) renamed /T24
- net Net-(RV7-Pad1) renamed /T28
- net Net-(RV7-Pad2) renamed /T26
- net Net-(RV8-Pad1) renamed /T5
- net Net-(RV8-Pad2) renamed /T19
- net Net-(RV9-Pad1) renamed /T4
- net Net-(RV9-Pad2) renamed /T18
- net Net-(SW1-Pad1) renamed /T31
- net Net-(SW1-Pad3) renamed /T30
- U1 pad 32: unconnected-(U1-Pad32) -> GND
