File: Teensy/PCB/ADSRModule/ADSR_Module.kicad_pcb (KiCad board)
At the start: 2 copper layers, 53.3 x 106.7 mm, 41 parts, among them J1 Power_Connector_2x3, SW1 Mode_Switch, U1 Teensy4.0

Commit message: Generated Gerbers
Other:
- board text added: "+"
- board text removed: "5v"
Changed lines of the file:
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@@
     (pad_to_mask_clearance 0)
     (pcbplotparams
-      (layerselection 0x0280000_7ffffffe)
+      (layerselection 0x02810fc_ffffffff)
       (disableapertmacros false)
-      (usegerberextensions false)
-      (usegerberattributes true)
-      (usegerberadvancedattributes true)
-      (creategerberjobfile true)
+      (usegerberextensions true)
+      (usegerberattributes false)
+      (usegerberadvancedattributes false)
+      (creategerberjobfile false)
       (svguseinch false)
       (svgprecision 6)
@@
       (psnegative false)
       (psa4output false)
-      (plotreference false)
+      (plotreference true)
       (plotvalue false)
       (plotinvisibletext false)
-      (sketchpadsonfab true)
-      (subtractmaskfromsilk false)
-      (outputformat 5)
+      (sketchpadsonfab false)
+      (subtractmaskfromsilk true)
+      (outputformat 1)
       (mirror false)
       (drillshape 0)
       (scaleselection 1)
-      (outputdirectory "./")
+      (outputdirectory "ADSR_Module_Gerber")
     )
   )
@@
   (gr_line (start 71.12 142.24) (end 71.12 35.56) (layer "User.2") (width 0.15))
   (gr_line (start 124.46 142.24) (end 71.12 142.24) (layer "User.2") (width 0.15))
-  (gr_text "5v" (at 89.535 130.175) (layer "B.SilkS")
-    (effects (font (size 1 1) (thickness 0.15)) (justify mirror))
+  (gr_text "+" (at 86.995 130.175) (layer "B.SilkS")
+    (effects (font (size 2 2) (thickness 0.3)) (justify mirror))
   )
   (segment (start 88.9 58.42) (end 83.82 53.34) (width 0.25) (layer "F.Cu") (net 1))
@@
   (segment (start 82.485 72.295) (end 82.485 72.325) (width 0.25) (layer "F.Cu") (net 19))
   (via (at 96.52 66.675) (size 0.8) (drill 0.4) (layers "F.Cu" "B.Cu") (net 19))
+  (segment (start 96.52 66.675) (end 97.155 66.675) (width 0.25) (layer "B.Cu") (net 19))
+  (segment (start 97.536 66.294) (end 97.536 58.166) (width 0.25) (layer "B.Cu") (net 19))
   (segment (start 96.52 56.515) (end 97.155 55.88) (width 0.25) (layer "B.Cu") (net 19))
-  (segment (start 96.52 66.675) (end 97.155 66.675) (width 0.25) (layer "B.Cu") (net 19))
+  (segment (start 99.06 55.88) (end 104.14 60.96) (width 0.25) (layer "B.Cu") (net 19))
   (segment (start 96.52 57.15) (end 96.52 56.515) (width 0.25) (layer "B.Cu") (net 19))
   (segment (start 97.155 55.88) (end 99.06 55.88) (width 0.25) (layer "B.Cu") (net 19))
-  (segment (start 97.79 66.04) (end 97.79 58.42) (width 0.25) (layer "B.Cu") (net 19))
-  (segment (start 99.06 55.88) (end 104.14 60.96) (width 0.25) (layer "B.Cu") (net 19))
-  (segment (start 97.79 58.42) (end 96.52 57.15) (width 0.25) (layer "B.Cu") (net 19))
-  (segment (start 97.155 66.675) (end 97.79 66.04) (width 0.25) (layer "B.Cu") (net 19))
+  (segment (start 97.155 66.675) (end 97.536 66.294) (width 0.25) (layer "B.Cu") (net 19))
+  (segment (start 97.536 58.166) (end 96.52 57.15) (width 0.25) (layer "B.Cu") (net 19))
   (segment (start 99.065 50.815) (end 96.52 48.27) (width 0.25) (layer "F.Cu") (net 20))
   (segment (start 96.52 48.26) (end 91.44 48.26) (width 0.25) (layer "F.Cu") (net 20))
@@
   (segment (start 116.84 78.105) (end 116.84 73.914) (width 0.25) (layer "B.Cu") (net 24))
   (segment (start 116.84 99.06) (end 116.84 102.87) (width 0.25) (layer "F.Cu") (net 25))
-  (segment (start 116.84 102.87) (end 99.06 120.65) (width 0.25) (layer "F.Cu") (net 25))
   (segment (start 120.65 80.01) (end 121.285 80.645) (width 0.25) (layer "F.Cu") (net 25))
+  (segment (start 99.568 120.142) (end 98.358 120.142) (width 0.25) (layer "F.Cu") (net 25))
+  (segment (start 98.358 120.142) (end 96.565 121.935) (width 0.25) (layer "F.Cu") (net 25))
+  (segment (start 121.285 94.615) (end 116.84 99.06) (width 0.25) (layer "F.Cu") (net 25))
+  (segment (start 116.84 102.87) (end 99.568 120.142) (width 0.25) (layer "F.Cu") (net 25))
   (segment (start 121.285 80.645) (end 121.285 94.615) (width 0.25) (layer "F.Cu") (net 25))
-  (segment (start 99.06 120.65) (end 97.79 120.65) (width 0.25) (layer "F.Cu") (net 25))
-  (segment (start 96.565 121.935) (end 97.79 120.71) (width 0.25) (layer "F.Cu") (net 25))
-  (segment (start 97.79 120.71) (end 97.79 120.65) (width 0.25) (layer "F.Cu") (net 25))
-  (segment (start 121.285 94.615) (end 116.84 99.06) (width 0.25) (layer "F.Cu") (net 25))
   (via (at 120.65 80.01) (size 0.8) (drill 0.4) (layers "F.Cu" "B.Cu") (net 25))
   (segment (start 120.65 80.01) (end 120.84 79.82) (width 0.25) (layer "B.Cu") (net 25))
