File: Teensy/PCB/USB_IOModule/USB_IOModule.kicad_pcb (KiCad board)
At the start: 2 copper layers, 55.9 x 106.7 mm, 101 parts, among them J1 USB_B, J2 USB_A, J3 Power_Connector_2x3, U1 SC16IS762IPW, U2 Teensy4.0, X1 XO53

Commit message: Replaced Schematic Lines with references
Connections:
- net /Audio_Input_Left/Signal renamed /T0
- net /Audio_Input_Right/Signal renamed /T7
- net /Audio_Output_Left/Signal renamed /T1
- net /Audio_Output_Right/Signal renamed /T8
- net /Channel_1_Mod_Input/Signal renamed /T28
- net /Channel_1_Mod_Output/Signal renamed /T29
- net /Channel_1_Pitch_Input/Signal renamed /T16
- net /Channel_1_Pitch_Output/Signal renamed /T17
- net /Channel_1_Trigger_Input/Signal renamed /RXB
- net /Channel_1_Trigger_Output/Signal renamed /T14
- net /Channel_2_Mod_Input/Signal renamed /T25
- net /Channel_2_Mod_Output/Signal renamed /T24
- net /Channel_2_Pitch_Input/Signal renamed /T21
- net /Channel_2_Pitch_Output/Signal renamed /T20
- net /Channel_2_Trigger_Input/Signal renamed /T15
- net /Channel_2_Trigger_Output/Signal renamed /TXB
- net /Clock_Output/Signal renamed /TXA
- net Net-(J2-Pad2) renamed /TD-
- net Net-(J2-Pad3) renamed /TD+
- net Net-(R2-Pad1) renamed /T4
- net Net-(R3-Pad1) renamed /T5
- net Net-(R4-Pad1) renamed /T6
- net Net-(R5-Pad1) renamed /T2
- net Net-(R6-Pad1) renamed /T9
- net Net-(RV1-Pad1) renamed /T32
- net Net-(RV1-Pad2) renamed /T23
- net Net-(RV2-Pad1) renamed /T33
- net Net-(RV2-Pad2) renamed /T22
- net Net-(RV3-Pad1) renamed /T30
- net Net-(RV3-Pad2) renamed /T19
- net Net-(RV4-Pad1) renamed /T31
- net Net-(RV4-Pad2) renamed /T18
- net Net-(U1-Pad10) renamed /T10
- net Net-(U1-Pad11) renamed /T11
- net Net-(U1-Pad12) renamed /T12
- net Net-(U1-Pad13) renamed /T13
