File: Teensy/PCB/VCAModule/VCAModule.kicad_pcb (KiCad board)
At the start: 2 copper layers, 45.7 x 106.7 mm, 51 parts, among them J1 Power_Connector_2x3, U1 Teensy4.0

Commit message: Replaced Schematic Lines with references
Connections:
- net /CV_Input_1/Signal renamed /T7
- net /CV_Input_2/Signal renamed /T16
- net /CV_Input_3/Signal renamed /T25
- net /VCA_1_Input/Signal renamed /T0
- net /VCA_1_Output/Signal renamed /T1
- net /VCA_1_Output/Switch renamed /T28
- net /VCA_2_Input/Signal renamed /T15
- net /VCA_2_Output/Signal renamed /T8
- net /VCA_2_Output/Switch renamed /T29
- net /VCA_3_Input/Signal renamed /T21
- net /VCA_3_Output/Signal renamed /T14
- net Net-(RV1-Pad1) renamed /T2
- net Net-(RV1-Pad2) renamed /T17
- net Net-(RV2-Pad1) renamed /T4
- net Net-(RV2-Pad2) renamed /T18
- net Net-(RV3-Pad1) renamed /T6
- net Net-(RV3-Pad2) renamed /T19
- net Net-(RV4-Pad1) renamed /T9
- net Net-(RV4-Pad2) renamed /T20
- net Net-(RV5-Pad1) renamed /T10
- net Net-(RV5-Pad2) renamed /T22
- net Net-(RV6-Pad1) renamed /T12
- net Net-(RV6-Pad2) renamed /T23
- net Net-(RV7-Pad1) renamed /T3
- net Net-(RV7-Pad2) renamed /T24
- net Net-(RV8-Pad1) renamed /T5
- net Net-(RV8-Pad2) renamed /T26
- net Net-(RV9-Pad1) renamed /T11
- net Net-(RV9-Pad2) renamed /T27
